File: hw/PicoDeck/PicoDeck.kicad_sch (KiCad schematic)
At the start: 0 parts

Commit message: schematics started
Parts:
- added A2: Clone_Pro_Mini_Socket_NoSPH, PCM_arduino-library:Clone_Pro_Mini_Socket_NoSPH, symbol PCM_arduino-library:Clone_Pro_Mini_Socket_NoSPH
- added J1: Conn_01x04, symbol Connector_Generic:Conn_01x04
- added J2, J3: Conn_01x05, symbol Connector_Generic:Conn_01x05
- added J4, J5, J6, J7: Conn_01x02, symbol Connector_Generic:Conn_01x02
- added R1, R2, R3, R4: 4.7k, Resistor_THT:R_Axial_DIN0207_L6.3mm_D2.5mm_P10.16mm_Horizontal, symbol PCM_SL_Resistors:4.7k
Connections:
- new net: J4.2 (Pin_2), R1.1
- new net: J5.2 (Pin_2), R2.1
- new net: J7.2 (Pin_2), R4.1
- new net: J6.2 (Pin_2), R3.1
- new net GND: J4.1 (Pin_1), J5.1 (Pin_1), J6.1 (Pin_1), J7.1 (Pin_1)
- new net VCC: R1.2, R2.2, R3.2, R4.2
